File: M_M-PCB/fulbo.kicad_sch (KiCad schematic)
At the start: 28 parts, among them J3 batt, J4 led rgb, J5 motor izq, J6 led rgb, J7 motor der, SW1 SW_SPDT, U1 ESP32s, U3 L7805, U4 L298(H)N

Commit message: xd
Parts:
- removed C2: 10uF, EESTN5:CAP_0.1, symbol Device:C_Polarized
- removed C3: 200uF, EESTN5:CAP_0.1, symbol Device:C_Polarized
- removed J4, J6: led rgb, EESTN5:pin_strip_4, symbol EESTN5:Conn_01x04
- removed R1: 1kohm, EESTN5:RES0.3, symbol EESTN5:R
- removed R2, R3, R4, R5, R6, R7: 100, EESTN5:RES0.3, symbol EESTN5:R
- removed U3: L7805, EESTN5:to220, symbol Regulator_Linear:L7805
- added C4: 100uF 25v, EESTN5:CAP_ELEC_5x11mm, symbol EESTN5:CAPAPOL
- added C5, C6: 100nF, EESTN5:CAP_0.1, symbol EESTN5:C
- added C7: 10uF 16v, EESTN5:CAP_ELEC_5x11mm, symbol EESTN5:CAPAPOL
- added D10: LED, symbol Device:LED
- added R1, R2: R, symbol Device:R
- added U2: L7805, EESTN5:TO-220, symbol Regulator_Linear:L7805
- D9: footprint EESTN5:Pin_Header_2 -> (none)
Connections:
- net +5V: now also C6.1, C7.1, U2.3 (OUT)
- net GND: now also C4.2, C5.2, C6.2, C7.2, D10.1 (K), U2.2 (GND)
- net VCC: now also C4.1, C5.1, U2.1 (IN)
- net at D9.2 (A): now also R1.2
- net pin_Blue renamed pin_A
- net pin_A: now also R1.1
- net pin_Green renamed pin_B
- net pin_B: now also R2.1
- net pin_Red: no longer names the net of U1.29 (IO5)
- new net: D10.2 (A), R2.2
